File: temperatureShield/Hardware/tempShield.brd (EAGLE design)
At the start: 160 x 100 mm, 4 parts

Commit message: still work on the schematic
Parts:
- removed LCD1: (no value), Particle:LCD
- added C1: 0.1uF, SparkFun-Capacitors:0603-CAP
- added J1: ADAFRUIT2_1X2-3.5MM, asset-tracker-v007:ADAFRUIT2_1X2-3.5MM
- added R1, R11, R2, R3, R4, R5, R6: 10k, SparkFun-Resistors:0603-RES
- added R10, R12, R13, R14, R15, R16, R7, R8, R9: 100K, programming-rig-v402:R0402
- added S1: (no value), Particle:TACTILE_SWITCH_SMD
- added U$1: MICROBUILDER_ELECTRON_SMT, asset-tracker-v007:MICROBUILDER_ELECTRON_SMT
- added U$2: PARTICLE-DEVICES_ELECTRON_WITH_STACKABLE_HEADERS, fuelview_v001:PARTICLE-DEVICES_ELECTRON_STACKABLE
- added U3: FUJITSU_MB85RS1MT, fuelview_v001:FUJITSU_SO08
- added U4: (no value), Particle:LCD
- U1: value (none) -> SHT30
- moved U$3 238.5 mm to (-88.9, -248.9)
- moved U1 72.3 mm to (-17.8, -50.8)
- moved U2 72.3 mm to (-16.5, -54.6)
Connections:
- new net !ALERT: R11.1, U2.C2
- new net !CS: R2.1, U3.1
- new net !HOLD: R4.1, U3.7
- new net +3V3: C1.2, R10.2, R11.2, R2.2, R3.2, R4.2, R5.2, R6.2, R7.2, R8.2, R9.2, U1.5, U2.A3, U3.8
- new net ALERT: R6.1, U1.3
- new net COM1: R10.1, R15.2, U4.1
- new net COM2: R14.2, R9.1, U4.2
- new net COM3: R13.2, R8.1, U4.3
- new net COM4: R12.2, R7.1, U4.4
- new net D0: U4.5
- new net D1: U4.6
- new net D2: U4.7
- new net D3: U4.8
- new net D4: U4.9
- new net D5: U4.10
- new net D6: U4.11
- new net D7: U4.12
- new net MISO: U3.2
- new net MOSI: U3.5
- new net N$2: R3.1, U3.3
- new net RESET: R5.1, U1.6
- new net SCK: U3.6
- new net SCL: U1.4, U2.B3
- new net SDA: U1.1, U2.C3
- new net VBAT: U$2.#34, U$2.34, U$2.@34
- net 3V3: now also U$1.1A, U$1.1B, U$2.#36, U$2.36, U$2.@36
- net GND: now also C1.1, R12.1, R13.1, R14.1, R15.1, U$1.29A, U$1.29B, U$1.30A, U$1.30B, U$2.#2, U$2.#33, U$2.2, U$2.33, U$2.@2, U$2.@33, U1.2, U1.7, U1.8, U1.9, U2.A1, U2.A2, U2.B1, U2.C1, U3.4
- net VIN: now also U$1.35A, U$1.35B, U$2.#1, U$2.1, U$2.@1

Commit message: finished the schematic and part of the layout
Parts:
- removed J1: ADAFRUIT2_1X2-3.5MM, asset-tracker-v007:ADAFRUIT2_1X2-3.5MM
- removed S1: (no value), Particle:TACTILE_SWITCH_SMD
- removed U$2: PARTICLE-DEVICES_ELECTRON_WITH_STACKABLE_HEADERS, fuelview_v001:PARTICLE-DEVICES_ELECTRON_STACKABLE
- removed U$3: ELECTRONDUALROW, Particle:ELECTRON_DUAL-ROW
- added C2, C3, C4, C5, C6: 0.1uF, SparkFun-Capacitors:0603-CAP
- added D1: (no value), SparkFun-LED:LED-0603
- added JP1: (no value), electron_v020:SPARKFUN-CONNECTORS_JST-2-SMD-VERT
- added R17, R18: 100K, programming-rig-v402:R0402
- added SW1: (no value), SparkFun-Electromechanical:TACTILE-SWITCH-SMD
- added U$4: MICROBUILDER_ELECTRON_SMT, asset-tracker-v007:MICROBUILDER_ELECTRON_SMT
- R1: value 10k -> 10K; device SparkFun-Resistors:0603-RES -> programming-rig-v402:R0402
- R16: value 100K -> 10K
- U$1: value MICROBUILDER_ELECTRON_SMT -> PARTICLE_DIODE_NT; device asset-tracker-v007:MICROBUILDER_ELECTRON_SMT -> electron_v020:PARTICLE_DIODE-DO-220AA_NT(SMP)
- U2: value (none) -> TMP007
- moved U$1 240.2 mm to (40.6, 44.5), flipped to the bottom, turned to 270 degrees
- moved R15 237.8 mm to (77.5, 34.3), flipped to the bottom, turned to 90 degrees
- moved R14 232.4 mm to (75.6, 34.3), flipped to the bottom, turned to 90 degrees
- moved R13 227.0 mm to (73.7, 34.3), flipped to the bottom, turned to 90 degrees
- moved R10 221.6 mm to (77.5, 36.8), flipped to the bottom, turned to 90 degrees
- moved R12 221.5 mm to (71.8, 34.3), flipped to the bottom, turned to 90 degrees
- moved R9 216.2 mm to (75.6, 36.8), flipped to the bottom, turned to 90 degrees
- moved R8 210.8 mm to (73.7, 36.8), flipped to the bottom, turned to 90 degrees
- moved R7 205.4 mm to (71.8, 36.8), flipped to the bottom, turned to 90 degrees
- moved R16 184.7 mm to (44.1, 31.0), flipped to the bottom, turned to 90 degrees
- moved R11 173.3 mm to (74.9, 40.0), flipped to the bottom, turned to 270 degrees
- moved R5 166.5 mm to (80.0, 40.0), flipped to the bottom, turned to 270 degrees
- moved R6 155.7 mm to (77.5, 40.0), flipped to the bottom, turned to 270 degrees
- moved U1 133.3 mm to (83.8, 35.6)
- moved U4 128.6 mm to (76.8, 31.1), turned to 180 degrees
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Connections:
- removed net 3V3: U$1.1A, U$1.1B, U$2.#36, U$2.36, U$2.@36, U$3.3V3, U$3.55, U$3.91
- removed net VBAT: U$2.#34, U$2.34, U$2.@34
- removed net VIN: U$1.35A, U$1.35B, U$2.#1, U$2.1, U$2.@1, U$3.1, U$3.37, U$3.VIN
- new net !WP: R3.1, U$4.12, U$4.12B, U3.3
- new net N$1: C6.2, U$1.CATHODE, U$4.1, U$4.1B
- new net N$10: U$4.5, U$4.5B
- new net N$11: U$4.6, U$4.6B
- new net N$12: U$4.18, U$4.18B
- new net N$3: JP1.VCC, U$1.ANODE
- new net N$4: R1.1, SW1.3, SW1.4, U$4.16, U$4.16B
- new net N$5: D1.C, R16.2
- new net N$6: U$4.35, U$4.35B
- new net N$7: U$4.34, U$4.34B
- new net N$8: U$4.3, U$4.3B
- new net N$9: U$4.4, U$4.4B
- net !ALERT: now also U$4.13, U$4.13B
- net !CS: now also U$4.10, U$4.10B
- net !HOLD: now also U$4.11, U$4.11B
- net +3V3: now also C2.2, C3.2, C4.2, C5.2, R1.2, R17.2, R18.2, U$4.36, U$4.36B
- net ALERT: now also U$4.14, U$4.14B
- net COM1: now also U$4.19, U$4.19B
- net COM2: now also U$4.20, U$4.20B
- net COM3: now also U$4.21, U$4.21B
- net COM4: now also U$4.22, U$4.22B
- net D0: now also U$4.25, U$4.25B
- net D1: now also U$4.26, U$4.26B
- net D2: now also U$4.27, U$4.27B
- net D3: now also U$4.28, U$4.28B
- net D4: now also U$4.29, U$4.29B
- net D5: now also U$4.30, U$4.30B
- net D6: now also U$4.31, U$4.31B
- net D7: now also U$4.32, U$4.32B
- net GND: now also C2.1, C3.1, C4.1, C5.1, C6.1, JP1.GND, R16.1, SW1.1, SW1.2, U$4.2, U$4.2B, U$4.33, U$4.33B; no longer U$1.29A, U$1.29B, U$1.30A, U$1.30B, U$2.#2, U$2.#33, U$2.2, U$2.33, U$2.@2, U$2.@33, U$3.2, U$3.38, U$3.58, U$3.94, U$3.GND, U$3.GND@2
- net MISO: now also U$4.8, U$4.8B
- net MOSI: now also U$4.7, U$4.7B
- net N$2: now also D1.A, U$4.17, U$4.17B; no longer R3.1, U3.3
- net RESET: now also U$4.15, U$4.15B
- net SCK: now also U$4.9, U$4.9B
- net SCL: now also R17.1, U$4.24, U$4.24B
- net SDA: now also R18.1, U$4.23, U$4.23B
Routing:
- net N$2: track 0.00 -> 57.1 mm, vias 0 -> 1
- net N$4: track 0.00 -> 55.1 mm, vias 0 -> 2
- net SCL: track 0.00 -> 40.9 mm, vias 0 -> 1
- net SDA: track 0.00 -> 38.5 mm, vias 0 -> 1
- net !ALERT: track 0.00 -> 34.2 mm, vias 0 -> 1
- net COM1: track 0.00 -> 29.0 mm, vias 0 -> 2
- net COM4: track 0.00 -> 27.6 mm, vias 0 -> 2
- net COM2: track 0.00 -> 26.8 mm, vias 0 -> 2
- net COM3: track 0.00 -> 26.5 mm, vias 0 -> 2
- net +3V3: track 0.00 -> 23.9 mm
- net !HOLD: track 0.00 -> 23.7 mm, vias 0 -> 2
- net SCK: track 0.00 -> 20.2 mm, vias 0 -> 2
- net GND: track 0.00 -> 19.9 mm
- net !WP: track 0.00 -> 18.8 mm, vias 0 -> 2
- net ALERT: track 0.00 -> 15.5 mm, vias 0 -> 1
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Other:
- board size 160 x 100 mm -> 57.1 x 31.8 mm

Commit message: Keep on the layout
Parts:
- moved D1 43.2 mm to (81.9, 36.3)
- moved R16 38.2 mm to (81.9, 36.3), turned to 270 degrees
- moved C2 5.98 mm to (89.9, 28.7), turned to 90 degrees
- moved U1 3.61 mm to (87.4, 36.2)
- moved R18 0.85 mm to (80.8, 31.8)
- moved R17 0.60 mm to (80.8, 33.6)
Routing:
- net SDA: track 38.5 -> 57.7 mm, vias 1 -> 2
- net SCL: track 40.9 -> 57.3 mm, vias 1 -> 2
- net ALERT: track 15.5 -> 28.8 mm
- net +3V3: track 23.9 -> 35.0 mm
- net N$5: track 8.43 -> 0.00 mm, vias 1 -> 0
- net N$2: track 57.1 -> 49.9 mm
- net RESET: track 13.8 -> 20.2 mm
Other:
- outline, holes or cut-outs redrawn

Commit message: update a little bit
Parts:
- moved JP1 2.22 mm to (38.5, 36.6)
- moved SW1 1.68 mm to (40.9, 36.2)
- moved C2 1.44 mm to (90.9, 29.7), turned to 0 degrees
- moved R1 1.35 mm to (44.0, 31.1)
Routing:
- net GND: track 19.9 -> 53.3 mm, vias 0 -> 5
- net RESET: track 20.2 -> 40.4 mm, vias 0 -> 1
- net +3V3: track 35.0 -> 50.1 mm, vias 0 -> 2
- net N$2: track 49.9 -> 56.0 mm
- net N$1: track 8.50 -> 11.2 mm
- net N$3: track 7.26 -> 9.23 mm
- net N$4: track 55.1 -> 57.0 mm
- net SDA: track 57.7 -> 59.4 mm, vias 2 -> 3
- net N$15: track 0.00 -> 1.60 mm
- net SCL: track 57.3 -> 58.4 mm, vias 2 -> 3
- net !ALERT: track 34.2 -> 35.3 mm, vias 1 -> 2
- net !CS: track 11.1 -> 11.7 mm

Commit message: UPATE A LITTLE BIT AGAIN
Parts:
- moved C3 5.24 mm to (48.5, 40.9), turned to 180 degrees
- moved C5 3.83 mm to (44.3, 31.4)
- moved C4 3.80 mm to (44.3, 30.3)
- moved R1 2.08 mm to (42.1, 30.3)
Routing:
- net !ALERT: track 35.3 -> 49.2 mm, vias 2 -> 3
- net N$4: track 57.0 -> 53.6 mm
- net SCL: track 58.4 -> 61.6 mm, vias 3 -> 4
- net SDA: track 59.4 -> 61.8 mm, vias 3 -> 4
- net +3V3: track 50.1 -> 48.0 mm
- net GND: track 53.3 -> 51.5 mm
- net N$15: track 1.60 -> 0.00 mm
- added copper zone on layer 1, net GND
- added copper zone on layer 16, net GND
- added copper zone on layer 1, net N$13
